File: eda/Light_Commander/analog.kicad_sch (KiCad schematic)
At the start: 32 parts, among them U2 TL084, U3 AD8544

Commit message: Power and UI on PCB
Connections:
- net +3V3A renamed +3V3
Changed lines of the file:
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@@
 			)
 		)
-		(property "Value" "+3V3A"
+		(property "Value" "+3V3"
 			(at 104.14 149.86 0)
 			(show_name no)
