File: eda/Light_Commander/analog.kicad_sch (KiCad schematic)
At the start: 32 parts, among them U2 TL084, U3 AD8544

Commit message: Add buttons, SWD, and LED reverse polarity protection to schematic
Other:
- note added: "CV Buffers, Gain, and Offset Scaling"
- note added: "Opamp Power Rails"
Changed lines of the file:
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@@
 	(generator_version "10.0")
 	(paper "A4")
+	(text "CV Buffers, Gain, and Offset Scaling"
+		(exclude_from_sim no)
+		(at 103.378 17.272 0)
+		(effects
+			(font
+				(size 1.905 1.905)
+			)
+			(justify left)
+		)
+	)
+	(text "Opamp Power Rails"
+		(exclude_from_sim no)
+		(at 73.152 144.272 0)
+		(effects
+			(font
+				(size 1.905 1.905)
+			)
+			(justify left)
+		)
+	)
 	(junction
 		(at 243.84 50.8)

Commit message: Fix footprints and finish first draft of schematic
Parts:
- C1, C2, C3, C4: footprint (none) -> Capacitor_SMD:C_0805_2012Metric
Changed lines of the file:
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@@
 			)
 		)
-		(property "Footprint" ""
+		(property "Footprint" "Capacitor_SMD:C_0805_2012Metric"
 			(at 92.4052 48.26 0)
 			(hide yes)
@@
 			)
 		)
-		(property "Footprint" ""
+		(property "Footprint" "Capacitor_SMD:C_0805_2012Metric"
 			(at 228.2952 48.26 0)
 			(hide yes)
@@
 			)
 		)
-		(property "Footprint" ""
+		(property "Footprint" "Capacitor_SMD:C_0805_2012Metric"
 			(at 94.9452 105.41 0)
 			(hide yes)
@@
 			)
 		)
-		(property "Footprint" ""
+		(property "Footprint" "Capacitor_SMD:C_0805_2012Metric"
 			(at 229.5652 104.14 0)
 			(hide yes)
