File: eda/Light_Commander/Light_Commander.kicad_sch (KiCad schematic)
At the start: 0 parts

Commit message: Power and UI on PCB
Parts:
- added J1: GATE0, footprints:PJ301M-12, symbol Connector_Audio:AudioJack2_Ground
- added J10: BUFFB, footprints:PJ301M-12, symbol Connector_Audio:AudioJack2_Ground
- added J11: BUFFC, footprints:PJ301M-12, symbol Connector_Audio:AudioJack2_Ground
- added J12: BUFFD, footprints:PJ301M-12, symbol Connector_Audio:AudioJack2_Ground
- added J2: GATE1, footprints:PJ301M-12, symbol Connector_Audio:AudioJack2_Ground
- added J3: GATE2, footprints:PJ301M-12, symbol Connector_Audio:AudioJack2_Ground
- added J4: GATE3, footprints:PJ301M-12, symbol Connector_Audio:AudioJack2_Ground
- added J5: INA, footprints:PJ301M-12, symbol Connector_Audio:AudioJack2_Ground
- added J6: INB, footprints:PJ301M-12, symbol Connector_Audio:AudioJack2_Ground
- added J7: INC, footprints:PJ301M-12, symbol Connector_Audio:AudioJack2_Ground
- added J8: IND, footprints:PJ301M-12, symbol Connector_Audio:AudioJack2_Ground
- added J9: BUFFA, footprints:PJ301M-12, symbol Connector_Audio:AudioJack2_Ground
Connections:
- net BUFFA_JACK: now also J9.T
- net BUFFB_JACK: now also J10.T
- net BUFFC_JACK: now also J11.T
- net BUFFD_JACK: now also J12.T
- net GND: now also J1.G, J1.S, J10.G, J11.G, J12.G, J2.G, J3.G, J4.G, J5.G, J5.S, J6.G, J7.G, J8.G, J9.G
- net INA_JACK: now also J5.T, J6.S
- net INB_JACK: now also J6.T, J7.S
- net INC_JACK: now also J7.T, J8.S
- net IND_JACK: now also J8.T
- new net GATE0_JACK: J1.T, J2.S
- new net GATE1_JACK: J2.T, J3.S
- new net GATE2_JACK: J3.T, J4.S
- new net GATE3_JACK: J4.T
- no-connect marks 0 -> 4
Other:
- added sheet Power (power.kicad_sch)
- added sheet UI (UI.kicad_sch)

Commit message: Voltage ref, BOOT0, and connections on PCB
Changed lines of the file:
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@@
 	(symbol
 		(lib_id "power:+2V5")
-		(at 215.9 105.41 0)
+		(at 203.2 105.41 0)
 		(unit 1)
 		(body_style 1)
@@
 		(fields_autoplaced yes)
 		(property "Reference" "#PWR021"
-			(at 215.9 109.22 0)
+			(at 203.2 109.22 0)
 			(hide yes)
 			(show_name no)
@@
 		)
 		(property "Value" "+12V"
-			(at 215.9 100.33 0)
+			(at 203.2 100.33 0)
 			(show_name no)
 			(do_not_autoplace no)
@@
 		)
 		(property "Footprint" ""
-			(at 215.9 105.41 0)
-			(hide yes)
-			(show_name no)
-			(do_not_autoplace no)
-			(effects
-				(font
-					(size 1.27 1.27)
-				)
-			)
-		)
-		(property "Datasheet" ""
-			(at 215.9 105.41 0)
+			(at 203.2 105.41 0)
+			(hide yes)
+			(show_name no)
+			(do_not_autoplace no)
+			(effects
+				(font
+					(size 1.27 1.27)
+				)
+			)
+		)
+		(property "Datasheet" ""
+			(at 203.2 105.41 0)
 			(hide yes)
 			(show_name no)
@@
 		)
 		(property "Description" "Power symbol creates a global label with name \"+2V5\""
-			(at 215.9 105.41 0)
+			(at 203.2 105.41 0)
 			(hide yes)
 			(show_name no)
@@
 	(symbol
 		(lib_id "power:-12V")
-		(at 215.9 110.49 180)
+		(at 203.2 110.49 180)
 		(unit 1)
 		(body_style 1)
@@
 		(fields_autoplaced yes)
 		(property "Reference" "#PWR022"
-			(at 215.9 106.68 0)
+			(at 203.2 106.68 0)
 			(hide yes)
 			(show_name no)
@@
 		)
 		(property "Value" "-12V"
-			(at 215.9 115.57 0)
+			(at 203.2 115.57 0)
 			(show_name no)
 			(do_not_autoplace no)
@@
 		)
 		(property "Footprint" ""
-			(at 215.9 110.49 0)
-			(hide yes)
-			(show_name no)
-			(do_not_autoplace no)
-			(effects
-				(font
-					(size 1.27 1.27)
-				)
-			)
-		)
-		(property "Datasheet" ""
-			(at 215.9 110.49 0)
+			(at 203.2 110.49 0)
+			(hide yes)
+			(show_name no)
+			(do_not_autoplace no)
+			(effects
+				(font
+					(size 1.27 1.27)
+				)
+			)
+		)
+		(property "Datasheet" ""
+			(at 203.2 110.49 0)
 			(hide yes)
 			(show_name no)
@@
 		)
 		(property "Description" "Power symbol creates a global label with name \"-12V\""
-			(at 215.9 110.49 0)
+			(at 203.2 110.49 0)
 			(hide yes)
 			(show_name no)
@@
 	(symbol
 		(lib_id "power:+2V5")
-		(at 224.79 105.41 0)
+		(at 219.71 105.41 0)
+		(unit 1)
+		(body_style 1)
+		(exclude_from_sim no)
+		(in_bom yes)
+		(on_board yes)
+		(in_pos_files yes)
+		(dnp no)
+		(fields_autoplaced yes)
+		(property "Reference" "#PWR067"
+			(at 219.71 109.22 0)
+			(hide yes)
+			(show_name no)
+			(do_not_autoplace no)
+			(effects
+				(font
+					(size 1.27 1.27)
+				)
+			)
+		)
+		(property "Value" "+5V"
+			(at 219.71 100.33 0)
+			(show_name no)
+			(do_not_autoplace no)
+			(effects
+				(font
+					(size 1.27 1.27)
+				)
+			)
+		)
+		(property "Footprint" ""
+			(at 219.71 105.41 0)
+			(hide yes)
+			(show_name no)
+			(do_not_autoplace no)
+			(effects
+				(font
+					(size 1.27 1.27)
+				)
+			)
+		)
+		(property "Datasheet" ""
+			(at 219.71 105.41 0)
+			(hide yes)
+			(show_name no)
+			(do_not_autoplace no)
+			(effects
+				(font
+					(size 1.27 1.27)
+				)
+			)
+		)
+		(property "Description" "Power symbol creates a global label with name \"+2V5\""
+			(at 219.71 105.41 0)
+			(hide yes)
+			(show_name no)
+			(do_not_autoplace no)
+			(effects
+				(font
+					(size 1.27 1.27)
+				)
+			)
+		)
+		(pin "1"
+		)
+		(instances
+			(project "Light_Commander"
+				(path "/dc725142-0bfd-4f8d-931f-2d32b87c7a54"
+					(reference "#PWR067")
+					(unit 1)
+				)
+			)
+		)
+	)
+	(symbol
+		(lib_id "power:+2V5")
+		(at 212.09 105.41 0)
 		(unit 1)
 		(body_style 1)
@@
 		(fields_autoplaced yes)
 		(property "Reference" "#PWR024"
-			(at 224.79 109.22 0)
+			(at 212.09 109.22 0)
 			(hide yes)
 			(show_name no)
@@
 		)
 		(property "Value" "+3V3"
-			(at 224.79 100.33 0)
+			(at 212.09 100.33 0)
 			(show_name no)
 			(do_not_autoplace no)
@@
 		)
 		(property "Footprint" ""
-			(at 224.79 105.41 0)
-			(hide yes)
-			(show_name no)
-			(do_not_autoplace no)
-			(effects
-				(font
-					(size 1.27 1.27)
-				)
-			)
-		)
-		(property "Datasheet" ""
-			(at 224.79 105.41 0)
+			(at 212.09 105.41 0)
+			(hide yes)
+			(show_name no)
+			(do_not_autoplace no)
+			(effects
+				(font
+					(size 1.27 1.27)
+				)
+			)
+		)
+		(property "Datasheet" ""
+			(at 212.09 105.41 0)
 			(hide yes)
 			(show_name no)
@@
 		)
 		(property "Description" "Power symbol creates a global label with name \"+2V5\""
-			(at 224.79 105.41 0)
+			(at 212.09 105.41 0)
 			(hide yes)
 			(show_name no)
@@
 	(symbol
 		(lib_id "power:+2V5")
-		(at 208.28 105.41 0)
+		(at 227.33 105.41 0)
 		(unit 1)
 		(body_style 1)
@@
 		(fields_autoplaced yes)
 		(property "Reference" "#PWR023"
-			(at 208.28 109.22 0)
+			(at 227.33 109.22 0)
 			(hide yes)
 			(show_name no)
@@
 		)
 		(property "Value" "+2V5"
-			(at 208.28 100.33 0)
+			(at 227.33 100.33 0)
 			(show_name no)
 			(do_not_autoplace no)
@@
 		)
 		(property "Footprint" ""
-			(at 208.28 105.41 0)
-			(hide yes)
-			(show_name no)
-			(do_not_autoplace no)
-			(effects
-				(font
-					(size 1.27 1.27)
-				)
-			)
-		)
-		(property "Datasheet" ""
-			(at 208.28 105.41 0)
+			(at 227.33 105.41 0)
+			(hide yes)
+			(show_name no)
+			(do_not_autoplace no)
+			(effects
+				(font
+					(size 1.27 1.27)
+				)
+			)
+		)
+		(property "Datasheet" ""
+			(at 227.33 105.41 0)
 			(hide yes)
 			(show_name no)
@@
 		)
 		(property "Description" "Power symbol creates a global label with name \"+2V5\""
-			(at 208.28 105.41 0)
+			(at 227.33 105.41 0)
 			(hide yes)
 			(show_name no)
@@
 	(symbol
 		(lib_id "power:GND")
-		(at 224.79 110.49 0)
+		(at 212.09 110.49 0)
 		(unit 1)
 		(body_style 1)
@@
 		(fields_autoplaced yes)
 		(property "Reference" "#PWR025"
-			(at 224.79 116.84 0)
+			(at 212.09 116.84 0)
 			(hide yes)
 			(show_name no)
@@
 		)
 		(property "Value" "GND"
-			(at 224.79 115.57 0)
+			(at 212.09 115.57 0)
 			(show_name no)
 			(do_not_autoplace no)
@@
 		)
 		(property "Footprint" ""
-			(at 224.79 110.49 0)
-			(hide yes)
-			(show_name no)
-			(do_not_autoplace no)
-			(effects
-				(font
-					(size 1.27 1.27)
-				)
-			)
-		)
-		(property "Datasheet" ""
-			(at 224.79 110.49 0)
+			(at 212.09 110.49 0)
+			(hide yes)
+			(show_name no)
+			(do_not_autoplace no)
+			(effects
+				(font
+					(size 1.27 1.27)
+				)
+			)
+		)
+		(property "Datasheet" ""
+			(at 212.09 110.49 0)
 			(hide yes)
 			(show_name no)
@@
 		)
 		(property "Description" "Power symbol creates a global label with name \"GND\" , ground"
-			(at 224.79 110.49 0)
-			(hide yes)
-			(show_name no)
+			(at 212.09 110.49 0)
+			(hide yes)
+			(show_name no)
