File: eda/Light_Commander/Light_Commander.kicad_pcb (KiCad board)
At the start: 2 copper layers, 111 x 132 mm, 163 parts, among them J1 GATE0, J10 BUFFB, J11 BUFFC, J12 BUFFD, J13 Eurorack_Power, J14 USB_C_Receptacle_USB2.0_16P, J15 Conn_01x05, J16 MIDI_IN, J17 MIDI_THRU, J18 Conn_01x03, J19 Conn_02x07_Odd_Even, J2 GATE1, J20 Conn_02x03_Odd_Even, J3 GATE2, J4 GATE3, J5 INA, J6 INB, J7 INC, J8 IND, J9 BUFFA, Q1 MMBT3904, Q2 MMBT3904, Q3 MMBT3904, Q4 MMBT3904, Q5 Q_PMOS_GSD, Q6 Q_NMOS_GSD, Q7 Q_PMOS_GDS, SW1 RotaryEncoder_Switch, SW2 SW_Push, SW3 SW_DPDT_x2, SW4 SW_DPDT_x2, U1 STM32F446RETx, U10 6N137, U11 NXU0101GW, U2 TL084, U3 AD8544, U4 R-785.0-0.5, U5 AP2112K-3.3, U6 USBLC6-2SC6, U7 2.5V Ref, U8 NXU0101GW, U9 SH1106_OLED, Y1 8 MHz

Commit message: Start of PCB
Parts:
- added N1: Housing, footprints:Light_Commander_Panel, F.Cu at (0.00, 0.00)
- C1, C10, C11, C12, C13, C14, C15, C16, C17, C18, C19, C2, C20, C21, C22, C23, C24, C25, C26, C27, C28, C29, C3, C30, C31, C32, C33, C34, C35, C36, C37, C38, C4, C5, C6, C7, C8, C9, D1, D10, D2, D3, D4, D5, D6, D7, D8, D9, F1, F2, F3, F4, F5, J13, J14, J18, J19, J20, L1, L2, L3, L4, Q1, Q2, Q3, Q4, Q5, Q6, Q7, R1, R10, R11, R12, R13, R14, R15, R16, R17, R18, R19, R2, R20, R21, R22, R23, R24, R25, R26, R27, R28, R29, R3, R30, R31, R32, R33, R34, R35, R36, R37, R38, R39, R4, R40, R41, R42, R43, R44, R45, R46, R47, R48, R49, R5, R50, R51, R52, R53, R54, R55, R56, R57, R58, R6, R7, R8, R9, SW2, SW3, SW4, U1, U10, U11, U2, U3, U4, U5, U6, U7, U8, Y1: moved to B.Cu
- moved J17 342.6 mm to (460.1, 62.6)
- moved J16 342.6 mm to (447.0, 62.6)
- moved J11 293.2 mm to (374.6, 92.3)
- moved J12 293.2 mm to (385.7, 92.3)
- moved J15 293.2 mm to (398.5, 91.6)
- moved J5 293.2 mm to (374.6, 64.2)
- moved J6 293.2 mm to (385.7, 64.2)
- moved J8 293.2 mm to (374.6, 78.2)
- moved J9 293.2 mm to (385.7, 78.2)
- moved SW1 293.2 mm to (392.3, 152.6)
- moved J10 293.2 mm to (363.6, 92.3)
- moved J7 293.2 mm to (363.6, 78.2)
- moved SW5 293.2 mm to (362.6, 114.2)
- moved SW6 293.2 mm to (362.6, 123.2)
- moved SW7 293.2 mm to (362.6, 132.3)
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Other:
- board size 111 x 132 mm -> 71 x 108 mm

Commit message: Start of PCB design
Parts:
- C30, L4, R39, R40: moved to F.Cu
- moved J17 339.7 mm to (125.4, 121.0), turned to 180 degrees
- moved J16 324.8 mm to (125.4, 108.0), turned to 180 degrees
- moved J9 316.0 mm to (74.6, 134.0), turned to 180 degrees
- moved J5 305.4 mm to (74.6, 121.0), turned to 180 degrees
- moved J6 303.7 mm to (87.3, 121.0), turned to 180 degrees
- moved SW6 289.5 mm to (74.6, 94.0)
- moved SW1 285.4 mm to (121.0, 64.0)
- moved J10 279.4 mm to (87.3, 134.0), turned to 180 degrees
- moved SW8 279.3 mm to (87.3, 94.0)
- moved J11 277.8 mm to (100.0, 134.0), turned to 180 degrees
- moved J12 276.1 mm to (112.7, 134.0), turned to 180 degrees
- moved J15 272.8 mm to (129.2, 135.0), turned to -90 degrees
- moved SW9 268.6 mm to (100.0, 94.0)
- moved J7 267.0 mm to (100.0, 121.0), turned to 180 degrees
- moved J8 265.4 mm to (112.7, 121.0), turned to 180 degrees
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