File: eda/Light_Commander/Light_Commander.kicad_pcb (KiCad board)
At the start: 6 copper layers, 71 x 108 mm, 164 parts, among them J1 GATE0, J10 BUFFB, J11 BUFFC, J12 BUFFD, J13 Eurorack_Power, J14 USB_C_Receptacle_USB2.0_16P, J15 Conn_01x05, J16 MIDI_IN, J17 MIDI_THRU, J18 Conn_01x03, J19 Conn_02x07_Odd_Even, J2 GATE1, J20 Conn_02x03_Odd_Even, J3 GATE2, J4 GATE3, J5 INA, J6 INB, J7 INC, J8 IND, J9 BUFFA, Q1 MMBT3904, Q2 MMBT3904, Q3 MMBT3904, Q4 MMBT3904, Q5 Q_PMOS_GSD, Q6 Q_NMOS_GSD, Q7 Q_PMOS_GDS, SW1 RotaryEncoder_Switch, SW2 SW_Push, SW3 SW_DPDT_x2, SW4 SW_DPDT_x2, U1 STM32F446RETx, U10 6N137, U11 NXU0101GW, U2 TL084, U3 AD8544, U4 R-785.0-0.5, U5 AP2112K-3.3, U6 USBLC6-2SC6, U7 2.5V Ref, U8 NXU0101GW, U9 SH1106_OLED, Y1 8 MHz

Commit message: Initial PCB review from Mylo
Parts:
- J14: moved to B.Cu
- R36, R37: moved to F.Cu
- moved C5 73.8 mm to (93.9, 143.6)
- moved R36 3.00 mm to (68.5, 68.5)
- moved R37 3.00 mm to (68.5, 65.5)
- moved R2 2.80 mm to (91.0, 147.8)
- moved R20 2.80 mm to (97.0, 147.8)
- moved F5 0.20 mm to (126.3, 105.9)
- moved J14 0.20 mm to (65.0, 67.4), turned to 90 degrees
- moved J19 0.20 mm to (69.7, 57.0)
- moved SW7 0.20 mm to (125.2, 94.0)
- moved J15 0.20 mm to (129.0, 135.0)
Connections:
- net Net-(J14-D+-PadA6) renamed /Digital/D+
- net Net-(J14-D--PadA7) renamed /Digital/D-
Routing:
- net Net-(Q7-D): track 80.2 -> 41.3 mm, vias 5 -> 18
- net +5V_LED: track 162.8 -> 133.1 mm, vias 7 -> 19
- net GND: track 222.6 -> 202.5 mm
- net Net-(J14-SHIELD): track 19.2 -> 2.01 mm
- net Net-(J15-Pin_1): track 69.7 -> 58.1 mm
- net Net-(U9-VCC): track 33.7 -> 22.7 mm
- net +12V: track 95.4 -> 89.3 mm
- net -12V: track 110.3 -> 105.7 mm
- net Net-(SW3A-C): track 35.7 -> 38.7 mm
- net Net-(D7-K): track 20.8 -> 23.7 mm
- net Net-(R20-Pad1): track 3.35 -> 6.15 mm
- net Net-(R2-Pad1): track 3.35 -> 6.15 mm
- net BUFFD_JACK: track 31.6 -> 34.4 mm
- net BUFFA_JACK: track 32.7 -> 35.5 mm
- net /Digital/D-: track 11.5 -> 9.01 mm, vias 1 -> 0
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- added copper zone on B.Cu, net +5V_LED
- added copper zone on F.Cu, net +5V_LED
- added copper zone on In2.Cu, net +5V_LED
- added copper zone on In3.Cu, net +5V_LED
- added copper zone on In4.Cu, net +5V_LED
- added copper zone on B.Cu, net Net-(Q7-D)
- added copper zone on F.Cu, net Net-(Q7-D)
- added copper zone on In2.Cu, net Net-(Q7-D)
- added copper zone on In3.Cu, net Net-(Q7-D)
- added copper zone on In4.Cu, net Net-(Q7-D)
Other:
- board size 71 x 108 mm -> 70.2 x 108 mm
