File: eda/Light_Commander/power.kicad_sch (KiCad schematic)
At the start: 18 parts, among them J13 Eurorack_Power, Q5 Q_PMOS_GSD, Q6 Q_NMOS_GSD, U4 R-785.0-0.5, U5 AP2112K-3.3, U7 2.5V Ref

Commit message: Add buttons, SWD, and LED reverse polarity protection to schematic
Other:
- note added: "2.5V Reference"
- note added: "3.3V Regulator"
- note added: "5V Regulator"
- note added: "Eurorack power, reverse polarity protection, and ESD protection"
Changed lines of the file:
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@@
 	(generator_version "10.0")
 	(paper "A4")
+	(text "5V Regulator"
+		(exclude_from_sim no)
+		(at 124.46 69.088 0)
+		(effects
+			(font
+				(size 1.905 1.905)
+			)
+			(justify left)
+		)
+	)
+	(text "2.5V Reference"
+		(exclude_from_sim no)
+		(at 85.852 117.094 0)
+		(effects
+			(font
+				(size 1.905 1.905)
+			)
+			(justify left)
+		)
+	)
+	(text "Eurorack power, reverse polarity protection, and ESD protection"
+		(exclude_from_sim no)
+		(at 28.702 60.706 0)
+		(effects
+			(font
+				(size 1.905 1.905)
+			)
+			(justify left)
+		)
+	)
+	(text "3.3V Regulator"
+		(exclude_from_sim no)
+		(at 167.64 70.612 0)
+		(effects
+			(font
+				(size 1.905 1.905)
+			)
+			(justify left)
+		)
+	)
 	(junction
 		(at 104.14 151.13)
