File: eda/Light_Commander/Light_Commander_panel.kicad_pcb (KiCad board)
At the start: 2 copper layers, 70.8 x 128.5 mm, 8 parts

Commit message: Start of PCB design
Parts:
- added ?: , , F.Cu at (125.4, 108.9)
- added ?: , , F.Cu at (87.3, 121.6)
- added ?: , , F.Cu at (100.0, 121.6)
- added ?: , , F.Cu at (87.3, 134.3)
- added ?: , , F.Cu at (112.7, 121.6)
- added ?: , , F.Cu at (74.6, 121.6)
- added ?: , , F.Cu at (100.0, 134.3)
- added ?: , , F.Cu at (74.6, 134.3)
- added ?: , , F.Cu at (112.7, 134.3)
- added ?: , , F.Cu at (125.4, 121.6)

Commit message: Initial component placement
Parts:
- moved ? 50.8 mm to (74.6, 108.0)
- moved ? 40.5 mm to (87.3, 108.0)
Changed lines of the file:
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@@
 	(footprint ""
 		(layer "F.Cu")
-		(at 125.4 121.6)
+		(at 87.3 108)
 		(property "Reference" ""
 			(at 0 0 0)
@@
 	(footprint ""
 		(layer "F.Cu")
-		(at 125.4 108.9)
-		(property "Reference" ""
-			(at 0 0 0)
+		(at 74.6 108)
+		(property "Reference" ""
+			(at 0 0 0)

Commit message: Initial PCB review from Mylo
Other:
- board text added: "Either add copper and remove to make texture or just add copper"
- board text added: "Exposed metal"
- board text added: "F.Cu + F.Mask"
- board text added: "silkscreen only"
