File: eda/Light_Commander/digital.kicad_sch (KiCad schematic)
At the start: 40 parts, among them J14 USB_C_Receptacle_USB2.0_16P, J18 Conn_01x03, SW2 SW_Push, U1 STM32F446RETx, U10 6N137, U11 NXU0101GW, U6 USBLC6-2SC6, U8 NXU0101GW, Y1 8 MHz

Commit message: Initial PCB review from Mylo
Connections:
- net D+: now reaches J14.A6 (D+), J14.B6 (D+), U6.3 (I/O2)
- net D-: now reaches J14.A7 (D-), J14.B7 (D-), U6.1 (I/O1)
Changed lines of the file:
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@@
+		)
+	)
+	(label "D+"
+		(at 55.88 156.21 0)
+		(effects
+			(font
+				(size 1.27 1.27)
+			)
+			(justify left bottom)
+		)
+	)
+	(label "D-"
+		(at 55.88 153.67 0)
+		(effects
+			(font
+				(size 1.27 1.27)
+			)
+			(justify left bottom)
 		)
 	)
